File: BTEMS PCB/BTEMS.brd (EAGLE design)
At the start: 50.8 x 63.5 mm, 22 parts

Commit message: v1.1 changes added
Parts:
- added EXHEADER_POW1: (no value), SparkFun-Connectors:1X02
- BAT_HEADER: device SparkFun-Connectors:1X02_2.54_SCREWTERM -> SparkFun-Connectors:SCREWTERMINAL-3.5MM-2
- R1: value R1 -> 24k
- R2: value R2 -> 30k
- moved BAT_HEADER 3.39 mm to (3.43, 14.7), turned to 90 degrees
- moved R_GLED 0.64 mm to (48.3, 18.4)
- moved R_RLED 0.64 mm to (46.1, 18.4)
- moved EXHEADER_A4-5 0.63 mm to (26.7, 4.45)
- moved S1 0.51 mm to (3.68, 26.7)
- moved EXHEADER_A6-7 0.51 mm to (43.2, 19.8)
- moved EXHEADER_A0-3 0.38 mm to (11.4, 28.3)
- moved EXHEADER_D2-9 0.38 mm to (11.4, 7.24)
Connections:
- net 3.3V: now also EXHEADER_POW1.2
- net BAT_IN: now also BAT_HEADER.2; no longer BAT_HEADER.P2
- net GND: now also BAT_HEADER.1, EXHEADER_POW1.1; no longer BAT_HEADER.P1
Routing:
- net SCL: track 151.9 -> 145.7 mm
- net N$3: track 3.43 -> 4.99 mm
- net A7: track 15.9 -> 17.2 mm
- net SDA: track 157.2 -> 156.1 mm
- net D9: track 15.7 -> 16.6 mm
- net A6: track 11.6 -> 12.3 mm
- net N$2: track 2.35 -> 2.98 mm
- net D11: track 33.1 -> 33.6 mm
Other:
- outline, holes or cut-outs redrawn
- board text added: "v1.1"
- board text removed: "v1.0"

Commit message: v1.1 final, mostly finished BOM
Parts:
- added EXHEADER2_A4_5: (no value), SparkFun-Connectors:1X02
- moved EXHEADER_POW1 5.08 mm to (26.7, 32.3), turned to 180 degrees
Connections:
- net SCL: now also EXHEADER2_A4_5.2
- net SDA: now also EXHEADER2_A4_5.1
Routing:
- net SDA: track 156.1 -> 170.6 mm, vias 1 -> 2
- net SCL: track 145.7 -> 160.0 mm, vias 1 -> 2
Other:
- outline, holes or cut-outs redrawn
Changed lines of the file:
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@@
 <wire x1="50.8" y1="63.5" x2="50.8" y2="0" width="0.4064" layer="20"/>
 <wire x1="50.8" y1="0" x2="0" y2="0" width="0.4064" layer="20"/>
-<wire x1="0" y1="0" x2="76.2" y2="0" width="0.4064" layer="49"/>
-<wire x1="76.2" y1="0" x2="76.2" y2="127" width="0.4064" layer="49"/>
-<wire x1="76.2" y1="127" x2="0" y2="127" width="0.4064" layer="49"/>
-<wire x1="0" y1="127" x2="0" y2="0" width="0.4064" layer="49"/>
 <wire x1="0" y1="12.7" x2="10.16" y2="12.7" width="0.4064" layer="21"/>
 <wire x1="10.16" y1="12.7" x2="10.16" y2="0" width="0.4064" layer="21"/>
@@
 <vertex x="40.64" y="56.261"/>
 </polygon>
-<text x="40.64" y="35.56" size="2.54" layer="21">v1.1</text>
+<text x="41.148" y="35.56" size="2.54" layer="21">v1.1</text>
 <text x="1.651" y="60.706" size="1.016" layer="21" rot="SR270">Environmental Fluid Dynamics Lab</text>
 <text x="6.35" y="55.245" size="3.81" layer="29" rot="SR270">BTEMS</text>
-<wire x1="7.62" y1="26.67" x2="7.62" y2="8.89" width="0.4064" layer="20"/>
-<text x="17.78" y="32.004" size="0.8128" layer="21">GND</text>
-<text x="25.908" y="32.004" size="0.8128" layer="21">3.3V</text>
+<wire x1="7.62" y1="26.67" x2="7.62" y2="8.89" width="0.4064" layer="25"/>
+<text x="25.654" y="29.972" size="0.8128" layer="21">GND</text>
+<text x="22.86" y="29.972" size="0.8128" layer="21">3.3V</text>
+<text x="20.574" y="29.972" size="0.8128" layer="27">SCL</text>
+<text x="18.034" y="29.972" size="0.8128" layer="27">SDA</text>
 </plain>
 <attributes>
@@
 </class>
 </classes>
-<designrules name="LaenPCBOrder">
+<designrules name="oshpark-2layer">
 <description language="de">&lt;b&gt;EAGLE Design Rules&lt;/b&gt;
 &lt;p&gt;
@@
 <param name="mvStopFrame" value="1"/>
 <param name="mvCreamFrame" value="0"/>
-<param name="mlMinStopFrame" value="3mil"/>
-<param name="mlMaxStopFrame" value="3mil"/>
+<param name="mlMinStopFrame" value="2.5mil"/>
+<param name="mlMaxStopFrame" value="2.5mil"/>
 <param name="mlMinCreamFrame" value="0mil"/>
 <param name="mlMaxCreamFrame" value="0mil"/>
@@
 <element name="SDSLOT" library="adafruit" package="06132" value="SDMMC06132" x="36.83" y="46.99" locked="yes" rot="R270"/>
 <element name="RTC_HEADER" library="SparkFun-Connectors" package="1X06_FEMALE_LOCK.010" value="" x="46.99" y="41.91" locked="yes" rot="R90"/>
-<element name="EXHEADER_POW1" library="SparkFun-Connectors" package="1X02" value="" x="21.59" y="32.385"/>
+<element name="EXHEADER_POW1" library="SparkFun-Connectors" package="1X02" value="" x="26.67" y="32.258" locked="yes" rot="R180"/>
+<element name="EXHEADER2_A4_5" library="SparkFun-Connectors" package="1X02" value="" x="19.05" y="32.258"/>
 </elements>
 <signals>
@@
 <wire x1="21.59" y1="20.32" x2="9.398" y2="20.32" width="0.4064" layer="16"/>
 <wire x1="9.398" y1="20.32" x2="6.985" y2="22.733" width="0.4064" layer="16"/>
-<wire x1="6.985" y1="22.733" x2="6.985" y2="51.435" width="0.4064" layer="16"/>
+<wire x1="6.985" y1="22.733" x2="6.985" y2="34.798" width="0.4064" layer="16"/>
+<wire x1="6.985" y1="34.798" x2="6.985" y2="51.435" width="0.4064" layer="16"/>
 <wire x1="6.985" y1="51.435" x2="10.16" y2="54.61" width="0.4064" layer="16"/>
 <wire x1="10.16" y1="54.61" x2="43.18" y2="54.61" width="0.4064" layer="16"/>
@@
 <wire x1="30.48" y1="5.588" x2="41.148" y2="5.588" width="0.4064" layer="1"/>
 <wire x1="41.148" y1="5.588" x2="41.402" y2="5.842" width="0.4064" layer="1"/>
-<wire x1="31.75" y1="2.667" x2="27.305" y2="2.667" width="0.4064" layer="1"/>
-<wire x1="27.305" y1="2.667" x2="26.924" y2="3.048" width="0.4064" layer="1"/>
 <wire x1="26.924" y1="3.048" x2="26.924" y2="4.3688" width="0.4064" layer="1"/>
 <wire x1="26.924" y1="4.3688" x2="26.8478" y2="4.445" width="0.4064" layer="1"/>
 <wire x1="19.05" y1="2.413" x2="26.289" y2="2.413" width="0.4064" layer="1"/>
 <wire x1="26.289" y1="2.413" x2="26.924" y2="3.048" width="0.4064" layer="1"/>
+<contactref element="EXHEADER2_A4_5" pad="1"/>
+<wire x1="19.05" y1="32.258" x2="19.05" y2="34.29" width="0.4064" layer="1"/>
+<wire x1="19.05" y1="34.29" x2="18.542" y2="34.798" width="0.4064" layer="1"/>
+<wire x1="18.542" y1="34.798" x2="6.985" y2="34.798" width="0.4064" layer="1"/>
+<via x="6.985" y="34.798" extent="1-16" drill="0.6" shape="square"/>
+<wire x1="26.924" y1="3.048" x2="27.559" y2="2.413" width="0.4064" layer="1"/>
+<wire x1="27.559" y1="2.413" x2="31.496" y2="2.413" width="0.4064" layer="1"/>
+<wire x1="31.496" y1="2.413" x2="31.75" y2="2.667" width="0.4064" layer="1"/>
 </signal>
 <signal name="SCL">
@@
 <wire x1="9.271" y1="22.479" x2="8.89" y2="22.86" width="0.4064" layer="1"/>
 <via x="8.89" y="22.86" extent="1-16" drill="0.6" shape="square"/>
-<wire x1="8.89" y1="22.86" x2="8.89" y2="51.435" width="0.4064" layer="16"/>
+<wire x1="8.89" y1="22.86" x2="8.89" y2="29.972" width="0.4064" layer="16"/>
+<wire x1="8.89" y1="29.972" x2="8.89" y2="51.435" width="0.4064" layer="16"/>
 <wire x1="8.89" y1="51.435" x2="10.16" y2="52.705" width="0.4064" layer="16"/>
 <wire x1="10.16" y1="52.705" x2="42.545" y2="52.705" width="0.4064" layer="16"/>
@@
 <wire x1="16.002" y1="4.572" x2="23.8252" y2="4.572" width="0.4064" layer="1"/>
 <wire x1="23.8252" y1="4.572" x2="23.9522" y2="4.445" width="0.4064" layer="1"/>
-<wire x1="34.29" y1="2.413" x2="34.29" y2="3.556" width="0.4064" layer="16"/>
-<wire x1="34.29" y1="3.556" x2="33.782" y2="4.064" width="0.4064" layer="16"/>
-<wire x1="33.782" y1="4.064" x2="30.48" y2="4.064" width="0.4064" layer="16"/>
-<wire x1="30.48" y1="4.064" x2="28.448" y2="2.032" width="0.4064" layer="16"/>
-<wire x1="28.448" y1="2.032" x2="24.384" y2="2.032" width="0.4064" layer="16"/>
-<wire x1="24.384" y1="2.032" x2="23.876" y2="2.54" width="0.4064" layer="16"/>
-<wire x1="23.876" y1="2.54" x2="23.876" y2="4.3688" width="0.4064" layer="16"/>
-<wire x1="23.876" y1="4.3688" x2="23.9522" y2="4.445" width="0.4064" layer="16"/>
 <wire x1="16.51" y1="2.667" x2="16.51" y2="4.064" width="0.4064" layer="1"/>
 <wire x1="16.51" y1="4.064" x2="16.002" y2="4.572" width="0.4064" layer="1"/>
+<contactref element="EXHEADER2_A4_5" pad="2"/>
+<wire x1="21.59" y1="32.258" x2="21.59" y2="30.988" width="0.4064" layer="1"/>
+<wire x1="21.59" y1="30.988" x2="21.082" y2="30.48" width="0.4064" layer="1"/>
+<wire x1="21.082" y1="30.48" x2="10.414" y2="30.48" width="0.4064" layer="1"/>
+<via x="10.414" y="30.48" extent="1-16" drill="0.6" shape="square"/>
+<wire x1="10.414" y1="30.48" x2="9.398" y2="30.48" width="0.4064" layer="16"/>
+<wire x1="9.398" y1="30.48" x2="8.89" y2="29.972" width="0.4064" layer="16"/>
+<wire x1="34.29" y1="2.413" x2="34.29" y2="3.81" width="0.4064" layer="16"/>
+<wire x1="34.29" y1="3.81" x2="33.782" y2="4.318" width="0.4064" layer="16"/>
+<wire x1="33.782" y1="4.318" x2="30.48" y2="4.318" width="0.4064" layer="16"/>
+<wire x1="30.48" y1="4.318" x2="28.448" y2="2.286" width="0.4064" layer="16"/>
+<wire x1="28.448" y1="2.286" x2="24.384" y2="2.286" width="0.4064" layer="16"/>
+<wire x1="24.384" y1="2.286" x2="24.13" y2="2.54" width="0.4064" layer="16"/>
+<wire x1="24.13" y1="2.54" x2="24.13" y2="4.2672" width="0.4064" layer="16"/>
+<wire x1="24.13" y1="4.2672" x2="23.9522" y2="4.445" width="0.4064" layer="16"/>
 </signal>
 <signal name="3.3V">
